File: Circuito/DomIO32.sch (KiCad schematic (older format))
At the start: 51 parts, among them J2 ICSP, J3 OSTTC032162, J4 OSTTC032162, J5 Conector2X5, SW1 TactSwitch, U1 LM1117-3.3, U2 PIC32MM0064GPL028-I-SO, U3 ESP-02, X1 X, X2 X, X3 X

Commit message: Correccion
Se agrega la conexion del pin 6 del modulo wifi
Parts:
- U2: symbol DomIO32:PIC32MM0064GPL028-I-SO -> DomIO32-rescue:PIC32MM0064GPL028-I-SO-DomIO32
- U3: symbol DomIO32:ESP-02 -> DomIO32-rescue:ESP-02-DomIO32
Connections:
- wire segments 195 -> 197
Other:
- moved on the sheet: C13
Changed lines of the file:
@@
 EESchema Schematic File Version 4
-LIBS:DomIO32-cache
-EELAYER 26 0
+EELAYER 30 0
 EELAYER END
 $Descr A4 11693 8268
@@
 $EndDescr
 $Comp
-L DomIO32:ESP-02 U3
+L DomIO32-rescue:ESP-02-DomIO32 U3
 U 1 1 5DCB6F71
 P 7050 1800
@@
 L Device:C C13
 U 1 1 5DCDBD3D
-P 7600 3150
-F 0 "C13" H 7250 3250 50  0000 L CNN
-F 1 "100nf / 50v" H 7000 3150 50  0000 L CNN
-F 2 "Capacitor_SMD:C_0805_2012Metric_Pad1.15x1.40mm_HandSolder" H 7638 3000 50  0001 C CNN
-F 3 "~" H 7600 3150 50  0001 C CNN
-	1    7600 3150
+P 7600 3050
+F 0 "C13" H 7250 3150 50  0000 L CNN
+F 1 "100nf / 50v" H 7000 3050 50  0000 L CNN
+F 2 "Capacitor_SMD:C_0805_2012Metric_Pad1.15x1.40mm_HandSolder" H 7638 2900 50  0001 C CNN
+F 3 "~" H 7600 3050 50  0001 C CNN
+	1    7600 3050
 	1    0    0    -1
 $EndComp
@@
 	7600 3550 7800 3550
 Connection ~ 7600 3550
-Wire Wire Line
-	7600 3550 7600 3300
-Wire Wire Line
-	7600 3000 7600 2850
 Connection ~ 7600 2750
 Connection ~ 5500 3200
@@
 Wire Wire Line
 	7800 2850 7600 2850
-Connection ~ 7600 2850
 Wire Wire Line
 	7600 2850 7600 2750
@@
 	8600 4050 9600 4050
 $Comp
-L DomIO32:PIC32MM0064GPL028-I-SO U2
+L DomIO32-rescue:PIC32MM0064GPL028-I-SO-DomIO32 U2
 U 1 1 5DD039C1
 P 3950 3450
@@
 Wire Wire Line
 	8600 4150 9650 4150
+Wire Wire Line
+	7600 3200 7600 3250
+Wire Wire Line
+	7600 2900 7600 2850
+Connection ~ 7600 2850
+Wire Wire Line
+	7800 3250 7600 3250
+Connection ~ 7600 3250
+Wire Wire Line
+	7600 3250 7600 3550
 $EndSCHEMATC

Commit message: Encapsulado PIC
Correcciones al encapsulado del PIC
Parts:
- U2: value PIC32MM0064GPL028-I-SO -> PIC32MM0064GPL028-I-SS
Changed lines of the file:
@@
 P 3950 3450
 F 0 "U2" H 4550 3415 50  0000 C CNN
-F 1 "PIC32MM0064GPL028-I-SO" H 4550 3324 50  0000 C CNN
+F 1 "PIC32MM0064GPL028-I-SS" H 4550 3324 50  0000 C CNN
 F 2 "Package_SO:SSOP-28_5.3x10.2mm_P0.65mm" H 3950 3300 50  0001 C CNN
 F 3 "" H 3950 3300 50  0001 C CNN

Commit message: update
update
Parts:
- removed J5: Conector2X5, Connector_Molex:Molex_Mini-Fit_Jr_5566-10A_2x05_P4.20mm_Vertical, symbol Connector_Generic:Conn_02x05_Odd_Even
- added J5: Conector 2x5, symbol Connector_Generic:Conn_02x05_Counter_Clockwise
- J2: value ICSP -> Conector 1x5
Connections:
- net +12V: now also J5.10 (Pin_10)
- net GND: now also J5.6 (Pin_6)
- net at R14.2: now also J5.4 (Pin_4)
- net at R15.2: now also J5.8 (Pin_8)
- net at R13.2: now also J5.1 (Pin_1)
- net at C12.1, D6.1 (K): now also J5.2 (Pin_2)
- net at R12.2: now also J5.3 (Pin_3)
- net at R11.2: now also J5.5 (Pin_5)
- net at R10.2: now also J5.7 (Pin_7)
- net at R9.2: now also J5.9 (Pin_9)
Other:
- moved on the sheet: C12, D6, R11, R12, R13
Changed lines of the file:
@@
 L power:GND #PWR018
 U 1 1 5DCD7E79
-P 9750 4300
-F 0 "#PWR018" H 9750 4050 50  0001 C CNN
-F 1 "GND" H 9755 4127 50  0001 C CNN
-F 2 "" H 9750 4300 50  0001 C CNN
-F 3 "" H 9750 4300 50  0001 C CNN
-	1    9750 4300
+P 9750 4800
+F 0 "#PWR018" H 9750 4550 50  0001 C CNN
+F 1 "GND" H 9755 4627 50  0001 C CNN
+F 2 "" H 9750 4800 50  0001 C CNN
+F 3 "" H 9750 4800 50  0001 C CNN
+	1    9750 4800
 	1    0    0    -1
 $EndComp
@@
 	9400 2750 9750 2750
 Connection ~ 9750 3800
-Wire Wire Line
-	9750 3800 9750 4300
 Wire Wire Line
 	7800 2750 7600 2750
@@
 	7450 2750 7600 2750
 $Comp
-L Connector_Generic:Conn_02x05_Odd_Even J5
-U 1 1 5DE6D22A
-P 7600 4950
-F 0 "J5" V 7500 4650 50  0000 R CNN
-F 1 "Conector2X5" V 7600 4650 50  0000 R CNN
-F 2 "Connector_Molex:Molex_Mini-Fit_Jr_5566-10A_2x05_P4.20mm_Vertical" H 7600 4950 50  0001 C CNN
-F 3 "~" H 7600 4950 50  0001 C CNN
-	1    7600 4950
-	0    -1   1    0
-$EndComp
-$Comp
 L Connector_Generic:Conn_01x05 J2
 U 1 1 5DE6D3C2
 P 3000 5950
-F 0 "J2" V 2873 5662 50  0000 R CNN
-F 1 "ICSP" V 3100 6000 50  0000 R CNN
+F 0 "J2" V 2950 6550 50  0000 R CNN
+F 1 "Conector 1x5" V 3050 6750 50  0000 R CNN
 F 2 "Connector_PinHeader_2.54mm:PinHeader_1x05_P2.54mm_Vertical" H 3000 5950 50  0001 C CNN
 F 3 "~" H 3000 5950 50  0001 C CNN
@@
 L Device:R R11
 U 1 1 5DE92402
+P 6550 5550
+F 0 "R11" V 6550 5550 50  0000 C CNN
+F 1 "1K" V 6600 5350 50  0000 C CNN
+F 2 "Resistor_SMD:R_0805_2012Metric_Pad1.15x1.40mm_HandSolder" V 6480 5550 50  0001 C CNN
+F 3 "~" H 6550 5550 50  0001 C CNN
+	1    6550 5550
+	0    -1   -1   0
+$EndComp
+$Comp
+L Device:R R12
+U 1 1 5DE92480
+P 6500 4750
+F 0 "R12" V 6500 4750 50  0000 C CNN
+F 1 "1K" V 6550 4550 50  0000 C CNN
+F 2 "Resistor_SMD:R_0805_2012Metric_Pad1.15x1.40mm_HandSolder" V 6430 4750 50  0001 C CNN
+F 3 "~" H 6500 4750 50  0001 C CNN
+	1    6500 4750
+	0    -1   -1   0
+$EndComp
+Wire Wire Line
+	5650 6100 5650 7100
+$Comp
+L Device:R R13
+U 1 1 5DF5D0E2
 P 6500 4450
-F 0 "R11" V 6500 4450 50  0000 C CNN
+F 0 "R13" V 6500 4450 50  0000 C CNN
 F 1 "1K" V 6550 4250 50  0000 C CNN
 F 2 "Resistor_SMD:R_0805_2012Metric_Pad1.15x1.40mm_HandSolder" V 6430 4450 50  0001 C CNN
@@
 $EndComp
 $Comp
-L Device:R R12
-U 1 1 5DE92480
-P 6500 4550
-F 0 "R12" V 6500 4550 50  0000 C CNN
-F 1 "1K" V 6550 4350 50  0000 C CNN
-F 2 "Resistor_SMD:R_0805_2012Metric_Pad1.15x1.40mm_HandSolder" V 6430 4550 50  0001 C CNN
-F 3 "~" H 6500 4550 50  0001 C CNN
-	1    6500 4550
-	0    -1   -1   0
-$EndComp
-Wire Wire Line
-	6650 4550 7500 4550
-Wire Wire Line
-	7500 4550 7500 4750
-Wire Wire Line
-	6650 4450 7600 4450
-Wire Wire Line
-	7600 4450 7600 4750
-Wire Wire Line
-	6650 4350 7700 4350
-Wire Wire Line
-	7700 4350 7700 4750
-Wire Wire Line
-	6650 4250 7800 4250
-Wire Wire Line
-	7800 4250 7800 4750
-Wire Wire Line
-	5650 6100 5650 7100
-$Comp
-L Device:R R13
-U 1 1 5DF5D0E2
-P 6500 4650
-F 0 "R13" V 6500 4650 50  0000 C CNN
-F 1 "1K" V 6550 4450 50  0000 C CNN
-F 2 "Resistor_SMD:R_0805_2012Metric_Pad1.15x1.40mm_HandSolder" V 6430 4650 50  0001 C CNN
-F 3 "~" H 6500 4650 50  0001 C CNN
-	1    6500 4650
-	0    -1   -1   0
-$EndComp
-$Comp
 L power:GND #PWR016
 U 1 1 5DF86986
-P 7600 6200
-F 0 "#PWR016" H 7600 5950 50  0001 C CNN
-F 1 "GND" H 7605 6027 50  0001 C CNN
-F 2 "" H 7600 6200 50  0001 C CNN
-F 3 "" H 7600 6200 50  0001 C CNN
-	1    7600 6200
+P 8700 6200
+F 0 "#PWR016" H 8700 5950 50  0001 C CNN
+F 1 "GND" H 8705 6027 50  0001 C CNN
+F 2 "" H 8700 6200 50  0001 C CNN
+F 3 "" H 8700 6200 50  0001 C CNN
+	1    8700 6200
 	1    0    0    -1
 $EndComp
@@
 L power:+4V #PWR015
 U 1 1 5DF9CD51
-P 7000 5700
-F 0 "#PWR015" H 7000 5550 50  0001 C CNN
-F 1 "+4V" H 7015 5873 50  0000 C CNN
-F 2 "" H 7000 5700 50  0001 C CNN
-F 3 "" H 7000 5700 50  0001 C CNN
-	1    7000 5700
+P 8300 5750
+F 0 "#PWR015" H 8300 5600 50  0001 C CNN
+F 1 "+4V" H 8315 5923 50  0000 C CNN
+F 2 "" H 8300 5750 50  0001 C CNN
+F 3 "" H 8300 5750 50  0001 C CNN
+	1    8300 5750
 	1    0    0    -1
 $EndComp
@@
 L power:+12V #PWR017
 U 1 1 5DF9D3DB
-P 8000 5250
-F 0 "#PWR017" H 8000 5100 50  0001 C CNN
-F 1 "+12V" H 8015 5423 50  0000 C CNN
-F 2 "" H 8000 5250 50  0001 C CNN
-F 3 "" H 8000 5250 50  0001 C CNN
-	1    8000 5250
+P 8600 4600
+F 0 "#PWR017" H 8600 4450 50  0001 C CNN
+F 1 "+12V" H 8450 4700 50  0000 C CNN
+F 2 "" H 8600 4600 50  0001 C CNN
+F 3 "" H 8600 4600 50  0001 C CNN
+	1    8600 4600
 	1    0    0    -1
 $EndComp
@@
 Wire Wire Line
 	1200 5000 1200 5150
-Text Label 8600 5000 0    50   ~ 0
+Text Label 9850 5200 0    50   ~ 0
 Expansion
-Text Label 8600 5100 0    50   ~ 0
+Text Label 9850 5300 0    50   ~ 0
 1)_Exp01
-Text Label 8600 5200 0    50   ~ 0
+Text Label 9850 5400 0    50   ~ 0
 2)_+3v3
-Text Label 8600 5300 0    50   ~ 0
+Text Label 9850 5500 0    50   ~ 0
 3)_Exp03
-Text Label 8600 5400 0    50   ~ 0
+Text Label 9850 5600 0    50   ~ 0
 4)_Exp04_(d0)
-Text Label 8600 5500 0    50   ~ 0
+Text Label 9850 5700 0    50   ~ 0
 5)_Exp05
-Text Label 8600 5600 0    50   ~ 0
+Text Label 9850 5800 0    50   ~ 0
 6)_Gnd
-Text Label 8600 5700 0    50   ~ 0
+Text Label 9850 5900 0    50   ~ 0
 7)_Exp07
-Text Label 8600 5800 0    50   ~ 0
+Text Label 9850 6000 0    50   ~ 0
 8)_Exp08_(d1)
-Text Label 8600 5900 0    50   ~ 0
+Text Label 9850 6100 0    50   ~ 0
 9)_Exp09
-Text Label 8550 6000 0    50   ~ 0
+Text Label 9800 6200 0    50   ~ 0
 10)_+12v
 Wire Notes Line
-	8550 4950 8550 6050
+	9800 5150 9800 6250
 Wire Notes Line
-	8600 6100 9100 6100
+	9850 6300 10350 6300
 Wire Notes Line
-	9150 6050 9150 4950
+	10400 6250 10400 5150
 Wire Notes Line
-	9100 4900 8600 4900
+	10350 5100 9850 5100
 Text Label 850  4150 0    50   ~ 0
 RESET
@@
 	1    0    0    -1
 $EndComp
-Text Label 7450 5050 0    50   ~ 0
+Text Label 8600 5050 0    50   ~ 0
 Expansion
 $Comp
@@
 $EndComp
 Wire Wire Line
-	6650 4650 7400 4650
-Wire Wire Line
-	7400 4650 7400 4750
-Wire Wire Line
-	6700 5350 7500 5350
-Wire Wire Line
-	7500 5350 7500 5250
-Wire Wire Line
-	7700 5450 7700 5250
-Wire Wire Line
-	8000 5250 8000 5300
-Wire Wire Line
-	8000 5300 7800 5300
-Wire Wire Line
-	7800 5300 7800 5250
-Wire Wire Line
-	6700 5450 7700 5450
-Wire Wire Line
 	3800 4550 3400 4550
 Wire Wire Line
@@
 L Device:C C12
 U 1 1 5DF3C419
-P 7400 5950
-F 0 "C12" H 7200 5850 50  0000 L CNN
-F 1 "100nf / 50v" H 6900 5750 50  0000 L CNN
-F 2 "Capacitor_SMD:C_0805_2012Metric_Pad1.15x1.40mm_HandSolder" H 7438 5800 50  0001 C CNN
-F 3 "~" H 7400 5950 50  0001 C CNN
-	1    7400 5950
-	1    0    0    -1
-$EndComp
-Wire Wire Line
-	7000 5700 7000 5750
-Wire Wire Line
-	7000 5750 7050 5750
-Wire Wire Line
-	7350 5750 7400 5750
-Wire Wire Line
-	7400 5750 7400 5800
-Wire Wire Line
-	7400 5250 7400 5750
-Connection ~ 7400 5750
-Wire Wire Line
-	7600 5250 7600 6150
-Wire Wire Line
-	7400 6100 7400 6150
-Wire Wire Line
-	7400 6150 7600 6150
-Connection ~ 7600 6150
-Wire Wire Line
-	7600 6150 7600 6200
+P 8700 6000
+F 0 "C12" H 8500 5900 50  0000 L CNN
+F 1 "100nf / 50v" H 8200 5800 50  0000 L CNN
+F 2 "Capacitor_SMD:C_0805_2012Metric_Pad1.15x1.40mm_HandSolder" H 8738 5850 50  0001 C CNN
+F 3 "~" H 8700 6000 50  0001 C CNN
+	1    8700 6000
+	1    0    0    -1
+$EndComp
+Wire Wire Line
+	8300 5750 8300 5800
+Wire Wire Line
+	8300 5800 8350 5800
+Wire Wire Line
+	8650 5800 8700 5800
+Wire Wire Line
+	8700 5800 8700 5850
+Connection ~ 8700 5800
+Wire Wire Line
+	8700 6150 8700 6200
 Wire Wire Line
 	5650 7100 5650 7200
@@
 L Device:D D6
 U 1 1 5EE1D796
-P 7200 5750
-F 0 "D6" H 7200 5850 50  0000 C CNN
-F 1 "M7" H 7200 5625 50  0000 C CNN
-F 2 "Diode_SMD:D_SMA" H 7200 5750 50  0001 C CNN
-F 3 "~" H 7200 5750 50  0001 C CNN
-	1    7200 5750
+P 8500 5800
+F 0 "D6" H 8500 5900 50  0000 C CNN
+F 1 "M7" H 8500 5675 50  0000 C CNN
+F 2 "Diode_SMD:D_SMA" H 8500 5800 50  0001 C CNN
+F 3 "~" H 8500 5800 50  0001 C CNN
+	1    8500 5800
 	-1   0    0    1
 $EndComp
@@
 Wire Wire Line
 	5550 5350 6400 5350
-Wire Wire Line
-	6350 4450 6050 4450
-Wire Wire Line
-	6050 4450 6050 5250
-Wire Wire Line
-	6050 5250 3450 5250
-Wire Wire Line
-	3450 5250 3450 4650
-Wire Wire Line
-	6350 4650 6000 4650
-Wire Wire Line
-	6000 4650 6000 4450
-Wire Wire Line
-	6000 4450 5300 4450
-Wire Wire Line
-	6350 4550 6150 4550
-Wire Wire Line
-	6150 4550 6150 4750
-Wire Wire Line
-	6150 4750 5300 4750
 Wire Wire Line
 	5900 4550 5750 4550
@@
 Wire Wire Line
 	7600 3250 7600 3550
+$Comp
+L Connector_Generic:Conn_02x05_Counter_Clockwise J5
+U 1 1 604E3439
+P 8800 5050
+F 0 "J5" V 8900 5650 50  0000 R CNN
+F 1 "Conector 2x5" V 8800 5900 50  0000 R CNN
+F 2 "" H 8800 5050 50  0001 C CNN
+F 3 "~" H 8800 5050 50  0001 C CNN
+	1    8800 5050
+	0    -1   -1   0
+$EndComp
+Wire Wire Line
+	8600 5300 8600 5250
+Wire Wire Line
+	9000 4750 9000 4700
+Wire Wire Line
+	8900 5350 8900 5250
+Wire Wire Line
+	6700 5350 8900 5350
+Wire Wire Line
+	8900 4350 8900 4750
+Wire Wire Line
+	6650 4350 8900 4350
+Wire Wire Line
+	8800 5400 8800 5250
+Wire Wire Line
+	8800 4650 8800 4750
+Wire Wire Line
+	6650 4250 8700 4250
+Wire Wire Line
+	8700 4250 8700 4750
+Text Label 2900 6100 0    50   ~ 0
+ICSP
+Wire Wire Line
+	9750 3800 9750 4700
+Wire Wire Line
+	9000 4700 9750 4700
+Connection ~ 9750 4700
+Wire Wire Line
+	9750 4700 9750 4800
+Wire Wire Line
+	7450 5400 8800 5400
+Wire Wire Line
+	9400 5450 9400 4650
+Wire Wire Line
+	9400 4650 8800 4650
+Wire Wire Line
+	6700 5450 9400 5450
+Wire Wire Line
+	8700 5250 8700 5800
+Wire Wire Line
+	8600 4600 8600 4750
+Wire Wire Line
+	6700 5550 9000 5550
+Wire Wire Line
+	9000 5250 9000 5550
+Wire Wire Line
+	6400 5550 3450 5550
+Wire Wire Line
+	3450 4650 3450 5550
+Wire Wire Line
+	5300 4450 6350 4450
+Wire Wire Line
+	6650 4450 7550 4450
+Wire Wire Line
+	7550 4450 7550 5300
+Wire Wire Line
+	7550 5300 8600 5300
+Wire Wire Line
+	6650 4750 7450 4750
+Wire Wire Line
+	7450 4750 7450 5400
+Wire Wire Line
+	5300 4750 6350 4750
 $EndSCHEMATC

Commit message: Se corrige capacitor electrolitico para nuevas librerias
Se corrige capacitor electrolitico para nuevas librerias
Parts:
- C10, C14, C3: symbol Device:CP -> Device:C_Polarized
Changed lines of the file:
@@
 $EndComp
 $Comp
-L Device:CP C10
+L Device:C_Polarized C10
 U 1 1 5DCB76F2
 P 5600 4550
@@
 	5150 7250 5150 7100
 $Comp
-L Device:CP C3
+L Device:C_Polarized C3
 U 1 1 5DD06DD2
 P 3600 1700
@@
 $EndComp
 $Comp
-L Device:CP C14
+L Device:C_Polarized C14
 U 1 1 5ED72089
 P 2500 1700

Commit message: Cambio de planes
Cambio de planes
Parts:
- removed C12: 100nf / 50v, Capacitor_SMD:C_0805_2012Metric_Pad1.15x1.40mm_HandSolder, symbol Device:C
- removed D6: M7, Diode_SMD:D_SMA, symbol Device:D
- removed J5: Conector 2x5, symbol Connector_Generic:Conn_02x05_Counter_Clockwise
- removed R10, R11, R12, R9: 1K, Resistor_SMD:R_0805_2012Metric_Pad1.15x1.40mm_HandSolder, symbol Device:R
- removed U2: PIC32MM0064GPL028-I-SS, Package_SO:SSOP-28_5.3x10.2mm_P0.65mm, symbol DomIO32-rescue:PIC32MM0064GPL028-I-SO-DomIO32
- removed X1, X2, X3: X, MountingHole:MountingHole_3.5mm_Pad, symbol Connector_Generic:Conn_01x01
- added C5, C7: 100nf / 50v, Capacitor_SMD:C_0805_2012Metric_Pad1.18x1.45mm_HandSolder, symbol Device:C
- added D10, D11, D8, D9: LL4148, Diode_SMD:D_SOD-128, symbol Device:D
- added D3: Led Amarillo, Diode_SMD:D_0805_2012Metric_Pad1.15x1.40mm_HandSolder, symbol Device:LED
- added J2, J7: Bornera x2, TerminalBlock_Phoenix:TerminalBlock_Phoenix_PT-1,5-2-5.0-H_1x02_P5.00mm_Horizontal, symbol Connector:Screw_Terminal_01x02
- added J5: USB_B_Micro, Connector_USB:USB_Micro-B_GCT_USB3076-30-A, symbol Connector:USB_B_Micro
- added J6: Bornera x3, TerminalBlock_Phoenix:TerminalBlock_Phoenix_PT-1,5-3-5.0-H_1x03_P5.00mm_Horizontal, symbol Connector:Screw_Terminal_01x03
- added K1, K2, K3, K4: FINDER-36.11, Relay_THT:Relay_SPDT_Finder_36.11, symbol Relay:FINDER-36.11
- added Q1, Q2, Q3, Q4: BC848, Package_TO_SOT_SMD:SOT-23, symbol Device:Q_NPN_BEC
- added R19, R20, R21, R22, R4, R7, R8: 1K, Resistor_SMD:R_0805_2012Metric_Pad1.20x1.40mm_HandSolder, symbol Device:R
- added U2: PIC32MM0256GPM028-I-SS, Package_SO:SSOP-28_5.3x10.2mm_P0.65mm, symbol DomIO32:PIC32MM0256GPM028-I-SS
- C1, C2: footprint Capacitor_SMD:C_0805_2012Metric_Pad1.15x1.40mm_HandSolder -> Capacitor_SMD:C_0805_2012Metric_Pad1.18x1.45mm_HandSolder
- C10: renamed from C6; footprint Capacitor_SMD:C_0805_2012Metric_Pad1.15x1.40mm_HandSolder -> Capacitor_SMD:C_0805_2012Metric_Pad1.18x1.45mm_HandSolder
- C11: renamed from C7; footprint Capacitor_SMD:C_0805_2012Metric_Pad1.15x1.40mm_HandSolder -> Capacitor_SMD:C_0805_2012Metric_Pad1.18x1.45mm_HandSolder
- C12: renamed from C8; footprint Capacitor_SMD:C_0805_2012Metric_Pad1.15x1.40mm_HandSolder -> Capacitor_SMD:C_0805_2012Metric_Pad1.18x1.45mm_HandSolder
- C13: renamed from C11; footprint Capacitor_SMD:C_0805_2012Metric_Pad1.15x1.40mm_HandSolder -> Capacitor_SMD:C_0805_2012Metric_Pad1.18x1.45mm_HandSolder
- C14: renamed from C13; footprint Capacitor_SMD:C_0805_2012Metric_Pad1.15x1.40mm_HandSolder -> Capacitor_SMD:C_0805_2012Metric_Pad1.18x1.45mm_HandSolder
- C3: renamed from C14; value 100uf / 16v -> 1000uf / 50v; footprint Capacitor_THT:CP_Radial_D6.3mm_P2.50mm -> Capacitor_THT:CP_Radial_D8.0mm_P5.00mm
- C4: renamed from C9; footprint Capacitor_SMD:C_0805_2012Metric_Pad1.15x1.40mm_HandSolder -> Capacitor_SMD:C_0805_2012Metric_Pad1.18x1.45mm_HandSolder
- C8: renamed from C4; footprint Capacitor_SMD:C_0805_2012Metric_Pad1.15x1.40mm_HandSolder -> Capacitor_SMD:C_0805_2012Metric_Pad1.18x1.45mm_HandSolder
- C9: renamed from C5; footprint Capacitor_SMD:C_0805_2012Metric_Pad1.15x1.40mm_HandSolder -> Capacitor_SMD:C_0805_2012Metric_Pad1.18x1.45mm_HandSolder
- D1: value Led Rojo -> Led Azul
- D5: renamed from D4; footprint Diode_SMD:D_0805_2012Metric_Pad1.15x1.40mm_HandSolder -> Diode_SMD:D_SOD-128
- D6: renamed from D5; value LL4148 -> M7; footprint Diode_SMD:D_0805_2012Metric_Pad1.15x1.40mm_HandSolder -> Diode_SMD:D_SMA
- J3, J4: value OSTTC032162 -> Bornera x3
- R1, R16, R17, R2, R3: footprint Resistor_SMD:R_0805_2012Metric_Pad1.15x1.40mm_HandSolder -> Resistor_SMD:R_0805_2012Metric_Pad1.20x1.40mm_HandSolder
- R10: renamed from R6; footprint Resistor_SMD:R_0805_2012Metric_Pad1.15x1.40mm_HandSolder -> Resistor_SMD:R_0805_2012Metric_Pad1.20x1.40mm_HandSolder
- R11: renamed from R7; footprint Resistor_SMD:R_0805_2012Metric_Pad1.15x1.40mm_HandSolder -> Resistor_SMD:R_0805_2012Metric_Pad1.20x1.40mm_HandSolder
- R12: renamed from R8; footprint Resistor_SMD:R_0805_2012Metric_Pad1.15x1.40mm_HandSolder -> Resistor_SMD:R_0805_2012Metric_Pad1.20x1.40mm_HandSolder
- R13, R14, R15: value 1K -> 22R; footprint Resistor_SMD:R_0805_2012Metric_Pad1.15x1.40mm_HandSolder -> Resistor_SMD:R_0805_2012Metric_Pad1.20x1.40mm_HandSolder
- R18: renamed from R19; footprint Resistor_SMD:R_0805_2012Metric_Pad1.15x1.40mm_HandSolder -> Resistor_SMD:R_0805_2012Metric_Pad1.20x1.40mm_HandSolder
- R5: renamed from R4; footprint Resistor_SMD:R_0805_2012Metric_Pad1.15x1.40mm_HandSolder -> Resistor_SMD:R_0805_2012Metric_Pad1.20x1.40mm_HandSolder
- R6: renamed from R18; footprint Resistor_SMD:R_0805_2012Metric_Pad1.15x1.40mm_HandSolder -> Resistor_SMD:R_0805_2012Metric_Pad1.20x1.40mm_HandSolder
- R9: renamed from R5; footprint Resistor_SMD:R_0805_2012Metric_Pad1.15x1.40mm_HandSolder -> Resistor_SMD:R_0805_2012Metric_Pad1.20x1.40mm_HandSolder
- renumbered C10 to C15, C3 to C6, D3 to D4, J2 to J1
Connections:
- net +12V: now also D10.1 (K), D11.1 (K), D9.1 (K), K2.A1, K3.A1, K4.A1; no longer C4.2, D4.2 (A), J4.1 (Pin_1)
- net GND: now also C5.1, C7.1, D3.1 (K), J2.2 (Pin_2), J5.5 (GND), Q1.2 (E), Q2.2 (E), Q3.2 (E), Q4.2 (E), U2.27 (AVss), U2.8 (Vss); no longer C14.2, J4.2 (Pin_2), U3.13 (GND), U3.18 (GND), U3.6 (IO15), U3.9 (GND)
- net at C15.1: now also U2.20 (Vcap)
- net at J1.1 (Pin_1), R5.1: now also U2.1 (MCLR)
- net at C13.1, D6.1 (K), J1.2 (Pin_2)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: now also U2.13 (Vdd), U2.28 (AVdd)
- net at R16.2: now also U2.26 (RP17/RB15)
- net at R17.2: now also U2.25 (RP16/RB14)
- net at C9.2, R9.1: now also U2.11 (SOSCI/RP10/RB4)
- net at C10.2, R10.1: now also U2.14 (PGED3/RP11/RB5)
- net at C11.2, R11.1: now also U2.16 (RP12/RB7)
- net at C12.2, R12.1: now also U2.17 (TCK/RP13/RB8)
- net at R14.1: now also U2.22 (D+/RB11)
- net at R2.2: now also U2.2 (PGEC2/RP1/RA0)
- net at R13.1: now also U2.21 (D-/RB10)
- net at R18.2: now also U2.24 (RP15/RB13)
- net at R3.2: now also U2.3 (PGED2/RP2/RA1)
- net at J1.4 (Pin_4): now also U2.4 (PGED1/RP6/RB0)
- net at J1.5 (Pin_5): now also U2.5 (PGEC1/RP7/RB1)
- net at R15.1: now also U2.15 (Vbus/RB6)
- net at R10.2: now also J4.1 (Pin_1); no longer J3.2 (Pin_2)
- net at R11.2: now also J4.2 (Pin_2); no longer J3.1 (Pin_1)
- net at C2.1, C3.1, D4.1 (K)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: now also D8.1 (K), K1.A1
- net at R14.2: now also J5.3 (D+)
- net at R15.2: now also J5.1 (VBUS)
- net at R13.2: now also J5.2 (D-)
- net +4V: no longer names the net of C6.1, C8.1, D6.2 (A), D7.2 (A), R6.1, U1.2 (VO)
- new net: C14.2, U3.13 (GND), U3.18 (GND), U3.6 (IO15), U3.9 (GND)
- new net: C4.2, D4.2 (A), J2.1 (Pin_1)
- new net: J3.1 (Pin_1), R7.2
- new net: J3.2 (Pin_2), R8.2
- new net: J7.1 (Pin_1), K1.11, K2.11, K3.11, K4.11
- new net: J6.3 (Pin_3), K1.14
- new net: D8.2 (A), K1.A2, Q1.3 (C)
- new net: D3.2 (A), R4.1
- new net: R4.2, U2.9 (OSC1/RP3/RA2)
- new net: J6.2 (Pin_2), K2.14
- new net: D9.2 (A), K2.A2, Q2.3 (C)
- new net: J6.1 (Pin_1), K3.14
- new net: D10.2 (A), K3.A2, Q3.3 (C)
- new net: J7.2 (Pin_2), K4.14
- new net: D11.2 (A), K4.A2, Q4.3 (C)
- new net: R22.1, U2.10 (OSC2/RP4/RA3)
- new net: Q4.1 (B), R22.2
- new net: R21.1, U2.12 (SOSCO/RP5/RA4)
- new net: Q3.1 (B), R21.2
- new net: R20.1, U2.18 (TMS/RP14/RB9)
- new net: Q2.1 (B), R20.2
- new net: R19.1, U2.19 (PGEC3/RP18/RC9)
- new net: Q1.1 (B), R19.2
- new net: C5.2, R7.1, U2.6 (RP8/RB2)
- new net: C7.2, R8.1, U2.7 (TDI/RP9/RB3)
Other:
- moved on the sheet: C1, C10, C11, C12, C13, C14, C15, C2, C3, C4, C6, C8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
