File: Circuito/DomIO32.sch (KiCad schematic (older format))
At the start: 67 parts, among them J1 Conector 1x5, J2 Bornera x2, J3 Bornera x3, J4 Bornera x3, J5 USB_B_Micro, J6 Bornera x3, J7 Bornera x2, K1 FINDER-36.11, K2 FINDER-36.11, K3 FINDER-36.11, K4 FINDER-36.11, Q1 BC848, Q2 BC848, Q3 BC848, Q4 BC848, SW1 TactSwitch, U1 LM1117-3.3, U2 PIC32MM0256GPM028-I-SS, U3 ESP-02

Commit message: Nuevo circuito co relees
Nuevo circuito co relees
Parts:
- added C16, C17: 100uf / 16v, Capacitor_THT:CP_Radial_D6.3mm_P2.50mm, symbol Device:C_Polarized
Connections:
- net GND: now also C17.2
- net at C14.1, D7.1 (K), U3.1 (Vdd)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: now also C16.1
- net at C14.2, U3.13 (GND), U3.18 (GND)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: now also C16.2
- net at C13.1, D6.1 (K), J1.2 (Pin_2)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: now also C17.1
Other:
- moved on the sheet: D7
Changed lines of the file:
@@
 U 1 1 5DCDBCE7
 P 5650 2550
-F 0 "C13" H 5765 2596 50  0000 L CNN
-F 1 "100nf / 50v" H 5765 2505 50  0000 L CNN
+F 0 "C13" H 5550 3000 50  0000 L CNN
+F 1 "100nf / 50v" H 5400 2900 50  0000 L CNN
 F 2 "Capacitor_SMD:C_0805_2012Metric_Pad1.18x1.45mm_HandSolder" H 5688 2400 50  0001 C CNN
 F 3 "~" H 5650 2550 50  0001 C CNN
@@
 U 1 1 5DCDBD3D
 P 6100 1300
-F 0 "C14" H 5750 1300 50  0000 L CNN
-F 1 "100nf / 50v" H 5550 1150 50  0000 L CNN
+F 0 "C14" H 6000 1900 50  0000 L CNN
+F 1 "100nf / 50v" H 5900 1800 50  0000 L CNN
 F 2 "Capacitor_SMD:C_0805_2012Metric_Pad1.18x1.45mm_HandSolder" H 6138 1150 50  0001 C CNN
 F 3 "~" H 6100 1300 50  0001 C CNN
@@
 Wire Wire Line
 	3700 1200 4100 1200
-Wire Wire Line
-	5950 1000 6100 1000
 $Comp
 L Connector_Generic:Conn_01x05 J1
@@
 Wire Wire Line
 	5150 3000 5650 3000
-$Comp
-L power:GND #PWR011
-U 1 1 5DDE0DA2
-P 5900 2850
-F 0 "#PWR011" H 5900 2600 50  0001 C CNN
-F 1 "GND" H 5905 2677 50  0001 C CNN
-F 2 "" H 5900 2850 50  0001 C CNN
-F 3 "" H 5900 2850 50  0001 C CNN
-	1    5900 2850
-	1    0    0    -1
-$EndComp
 Wire Wire Line
 	5350 2350 5650 2350
 Wire Wire Line
 	5650 2350 5650 2400
-Wire Wire Line
-	5650 2700 5650 2800
-Wire Wire Line
-	5900 2850 5900 2800
-Wire Wire Line
-	5900 2800 5650 2800
-Connection ~ 5650 2800
-Wire Wire Line
-	5650 2800 5650 3000
 $Comp
 L Device:C C4
@@
 L Device:D D7
 U 1 1 5EE1D488
-P 5800 1000
-F 0 "D7" H 5900 900 50  0000 C CNN
-F 1 "M7" H 5700 900 50  0000 C CNN
-F 2 "Diode_SMD:D_SMA" H 5800 1000 50  0001 C CNN
-F 3 "~" H 5800 1000 50  0001 C CNN
-	1    5800 1000
+P 5650 1000
+F 0 "D7" H 5750 900 50  0000 C CNN
+F 1 "M7" H 5550 900 50  0000 C CNN
+F 2 "Diode_SMD:D_SMA" H 5650 1000 50  0001 C CNN
+F 3 "~" H 5650 1000 50  0001 C CNN
+	1    5650 1000
 	-1   0    0    1
 $EndComp
@@
 	2000 3650 2000 3600
 Wire Wire Line
-	5650 1000 5350 1000
-Wire Wire Line
 	5150 3100 6300 3100
 Wire Wire Line
@@
 Wire Wire Line
 	4100 1000 4100 1200
-Connection ~ 5350 1000
 Connection ~ 4100 1200
 $Comp
@@
 	8400 600  2250 600
 Wire Wire Line
-	2200 2350 2750 2350
-Wire Wire Line
 	2250 600  2250 1200
 Wire Wire Line
@@
 Wire Wire Line
 	2000 2350 2750 2350
+$Comp
+L Device:C_Polarized C16
+U 1 1 62189655
+P 5850 1300
+F 0 "C16" H 5600 1150 50  0000 L CNN
+F 1 "100uf / 16v" H 5450 1000 50  0000 L CNN
+F 2 "Capacitor_THT:CP_Radial_D6.3mm_P2.50mm" H 5888 1150 50  0001 C CNN
+F 3 "~" H 5850 1300 50  0001 C CNN
+	1    5850 1300
+	1    0    0    -1
+$EndComp
+Wire Wire Line
+	5500 1000 5350 1000
+Connection ~ 5350 1000
+Wire Wire Line
+	5800 1000 5850 1000
+Wire Wire Line
+	5850 1150 5850 1000
+Connection ~ 5850 1000
+Wire Wire Line
+	5850 1000 6100 1000
+Wire Wire Line
+	5850 1450 5850 1500
+Wire Wire Line
+	5850 1500 6100 1500
+Wire Wire Line
+	5650 2700 5650 3000
+Wire Wire Line
+	5650 3000 5900 3000
+Wire Wire Line
+	6650 3000 6650 3700
+Connection ~ 5650 3000
+Connection ~ 6650 3700
+$Comp
+L Device:C_Polarized C17
+U 1 1 6221BD48
+P 5900 2550
+F 0 "C17" H 6000 2400 50  0000 L CNN
+F 1 "100uf / 16v" H 5700 2200 50  0000 L CNN
+F 2 "Capacitor_THT:CP_Radial_D6.3mm_P2.50mm" H 5938 2400 50  0001 C CNN
+F 3 "~" H 5900 2550 50  0001 C CNN
+	1    5900 2550
+	1    0    0    -1
+$EndComp
+Wire Wire Line
+	5650 2350 5900 2350
+Wire Wire Line
+	5900 2350 5900 2400
+Connection ~ 5650 2350
+Wire Wire Line
+	5900 2700 5900 3000
+Connection ~ 5900 3000
+Wire Wire Line
+	5900 3000 6650 3000
 $EndSCHEMATC

Commit message: Reestructuracion del proyecto
Reestructuracion del proyecto
Parts:
- removed J5: USB_B_Micro, Connector_USB:USB_Micro-B_GCT_USB3076-30-A, symbol Connector:USB_B_Micro
- removed R15: 22R, Resistor_SMD:R_0805_2012Metric_Pad1.20x1.40mm_HandSolder, symbol Device:R
- added J5: Conn_01x03, Connector_PinHeader_2.54mm:PinHeader_1x03_P2.54mm_Vertical, symbol Connector_Generic:Conn_01x03
- renumbered C16 to C14, C17 to C15, C14 to C16, C15 to C17, R14 to R13, R13 to R14, R16 to R15, R17 to R16, R18 to R17, R19 to R18, R20 to R19, R21 to R20, R22 to R21
Connections:
- net GND: now also J5.1 (Pin_1)
- net at R4.2: now also U2.12 (SOSCO/RP5/RA4); no longer U2.9 (OSC1/RP3/RA2)
- net at R21.1: now also U2.18 (TMS/RP14/RB9); no longer U2.10 (OSC2/RP4/RA3)
- net at R20.1: now also U2.19 (PGEC3/RP18/RC9); no longer U2.12 (SOSCO/RP5/RA4)
- net at R19.1: now also U2.21 (D-/RB10); no longer U2.18 (TMS/RP14/RB9)
- net at R18.1: now also U2.22 (D+/RB11); no longer U2.19 (PGEC3/RP18/RC9)
- net at R14.1: now also U2.9 (OSC1/RP3/RA2); no longer U2.21 (D-/RB10)
- net at R13.1: now also U2.10 (OSC2/RP4/RA3); no longer U2.22 (D+/RB11)
- net at R14.2: now also J5.2 (Pin_2)
- net at R13.2: now also J5.3 (Pin_3)
Other:
- note added: "Gnd"
- note added: "Rx"
- note added: "TX"
- moved on the sheet: R13, R14
