File: Circuito/DomIO32.kicad_pcb (KiCad board)
At the start: 2 copper layers, 50 x 50 mm, 51 parts, among them J2 ICSP, J3 OSTTC032162, J4 OSTTC032162, J5 Conector2X5, SW1 TactSwitch, U1 LM1117-3.3, U2 PIC32MM0064GPL028-I-SO, U3 ESP-02, X1 X, X2 X, X3 X

Commit message: Cambio de planes
Cambio de planes
Parts:
- removed X1, X2, X3: X, MountingHole:MountingHole_3.5mm_Pad
- added C15: 100uf / 16v, Capacitor_THT:CP_Radial_D6.3mm_P2.50mm, F.Cu at (90.0, 97.0)
- added D10: LL4148, Diode_SMD:D_SOD-128, F.Cu at (162.0, 76.0)
- added D11: LL4148, Diode_SMD:D_SOD-128, F.Cu at (178.0, 76.0)
- added D8: LL4148, Diode_SMD:D_SOD-128, F.Cu at (130.0, 76.0)
- added D9: LL4148, Diode_SMD:D_SOD-128, F.Cu at (146.0, 76.0)
- added J1: Conector 1x5, Connector_PinHeader_2.54mm:PinHeader_1x05_P2.54mm_Vertical, F.Cu at (110.0, 128.0)
- added J6: Bornera x3, TerminalBlock_Phoenix:TerminalBlock_Phoenix_PT-1,5-3-5.0-H_1x03_P5.00mm_Horizontal, F.Cu at (172.0, 48.0)
- added J7: Bornera x2, TerminalBlock_Phoenix:TerminalBlock_Phoenix_PT-1,5-2-5.0-H_1x02_P5.00mm_Horizontal, F.Cu at (182.0, 48.0)
- added K1: FINDER-36.11, Relay_THT:Relay_SPDT_Finder_36.11, F.Cu at (130.0, 71.0)
- added K2: FINDER-36.11, Relay_THT:Relay_SPDT_Finder_36.11, F.Cu at (146.0, 71.0)
- added K3: FINDER-36.11, Relay_THT:Relay_SPDT_Finder_36.11, F.Cu at (162.0, 71.0)
- added K4: FINDER-36.11, Relay_THT:Relay_SPDT_Finder_36.11, F.Cu at (178.0, 71.0)
- added Q1: BC848, Package_TO_SOT_SMD:SOT-23, F.Cu at (200.0, 106.0)
- added Q2: BC848, Package_TO_SOT_SMD:SOT-23, F.Cu at (200.0, 100.0)
- added Q3: BC848, Package_TO_SOT_SMD:SOT-23, F.Cu at (194.0, 100.0)
- added Q4: BC848, Package_TO_SOT_SMD:SOT-23, F.Cu at (194.0, 106.0)
- added R20: 1K, Resistor_SMD:R_0805_2012Metric_Pad1.20x1.40mm_HandSolder, F.Cu at (175.8, 133.6)
- added R21: 1K, Resistor_SMD:R_0805_2012Metric_Pad1.20x1.40mm_HandSolder, F.Cu at (189.5, 143.8)
- added R22: 1K, Resistor_SMD:R_0805_2012Metric_Pad1.20x1.40mm_HandSolder, F.Cu at (134.0, 143.0)
- C1, C11, C12, C13, C4, C5, C7, C8, C9: footprint Capacitor_SMD:C_0805_2012Metric_Pad1.15x1.40mm_HandSolder -> Capacitor_SMD:C_0805_2012Metric_Pad1.18x1.45mm_HandSolder
- C10, C14: value 100uf / 16v -> 100nf / 50v; footprint Capacitor_THT:CP_Radial_D6.3mm_P2.50mm -> Capacitor_SMD:C_0805_2012Metric_Pad1.18x1.45mm_HandSolder; moved to F.Cu
- C2: footprint Capacitor_SMD:C_0805_2012Metric_Pad1.15x1.40mm_HandSolder -> Capacitor_SMD:C_0805_2012Metric_Pad1.18x1.45mm_HandSolder; moved to B.Cu
- C3: value 100uf / 16v -> 1000uf / 50v; footprint Capacitor_THT:CP_Radial_D6.3mm_P2.50mm -> Capacitor_THT:CP_Radial_D8.0mm_P5.00mm; moved to F.Cu
- C6: value 100nf / 50v -> 100uf / 16v; footprint Capacitor_SMD:C_0805_2012Metric_Pad1.15x1.40mm_HandSolder -> Capacitor_THT:CP_Radial_D6.3mm_P2.50mm
- D1: value Led Rojo -> Led Azul; moved to F.Cu
- D2, SW1: moved to F.Cu
- D3: value M7 -> Led Amarillo; footprint Diode_SMD:D_SMA -> Diode_SMD:D_0805_2012Metric_Pad1.15x1.40mm_HandSolder
- D4: value LL4148 -> M7; footprint Diode_SMD:D_0805_2012Metric_Pad1.15x1.40mm_HandSolder -> Diode_SMD:D_SMA
- D5: footprint Diode_SMD:D_0805_2012Metric_Pad1.15x1.40mm_HandSolder -> Diode_SMD:D_SOD-128
- J2: value ICSP -> Bornera x2; footprint Connector_PinHeader_2.54mm:PinHeader_1x05_P2.54mm_Vertical -> TerminalBlock_Phoenix:TerminalBlock_Phoenix_PT-1,5-2-5.0-H_1x02_P5.00mm_Horizontal; moved to F.Cu
- J3, J4: value OSTTC032162 -> Bornera x3; moved to F.Cu
- J5: value Conector2X5 -> USB_B_Micro; footprint Connector_Molex:Molex_Mini-Fit_Jr_5566-10A_2x05_P4.20mm_Vertical -> Connector_USB:USB_Micro-B_GCT_USB3076-30-A; moved to F.Cu
- R1, R10, R11, R12, R16, R17, R18, R19, R2, R3, R4, R5, R6, R7, R8, R9: footprint Resistor_SMD:R_0805_2012Metric_Pad1.15x1.40mm_HandSolder -> Resistor_SMD:R_0805_2012Metric_Pad1.20x1.40mm_HandSolder
- R13, R14, R15: value 1K -> 22R; footprint Resistor_SMD:R_0805_2012Metric_Pad1.15x1.40mm_HandSolder -> Resistor_SMD:R_0805_2012Metric_Pad1.20x1.40mm_HandSolder
- U2: value PIC32MM0064GPL028-I-SO -> PIC32MM0256GPM028-I-SS; moved to B.Cu
- U3: moved to B.Cu
- moved C10 99.8 mm to (197.9, 121.5), turned to 0 degrees
- moved R2 98.4 mm to (193.6, 135.0), turned to 0 degrees
- moved C14 98.2 mm to (189.9, 126.0), turned to 0 degrees
- moved C4 94.0 mm to (194.7, 126.0), turned to 0 degrees
- moved C11 91.9 mm to (188.8, 133.5), turned to 0 degrees
- moved C13 86.6 mm to (189.9, 129.0), turned to 0 degrees
- moved R13 84.8 mm to (198.3, 132.0)
- moved R18 84.8 mm to (172.2, 136.8), turned to 0 degrees
- moved R3 78.3 mm to (175.8, 130.7), turned to 0 degrees
- moved R15 75.3 mm to (193.6, 137.9), turned to 0 degrees
- moved D6 73.0 mm to (195.0, 58.0), turned to 0 degrees
- moved D7 70.3 mm to (197.2, 86.0), turned to 0 degrees
- moved R4 69.5 mm to (156.6, 137.9)
- moved R17 68.8 mm to (189.5, 140.9), turned to 0 degrees
- moved R19 67.5 mm to (151.8, 140.9), turned to 0 degrees
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Connections:
- C10 pad 1: Net-(C10-Pad1) -> GND
- C10 pad 2: GND -> Net-(C10-Pad2)
- C11 pad 1: Net-(C11-Pad1) -> GND
- C11 pad 2: GND -> Net-(C11-Pad2)
- C12 pad 1: Net-(C12-Pad1) -> GND
- C12 pad 2: GND -> Net-(C12-Pad2)
- C14 pad 2: GND -> Net-(C14-Pad2)
- C2 pad 1: Net-(C14-Pad1) -> Net-(C2-Pad1)
- C3 pad 1: +4V -> Net-(C2-Pad1)
- C4 pad 1: +4V -> GND
- C4 pad 2: GND -> Net-(C4-Pad2)
- C6 pad 1: GND -> Net-(C6-Pad1)
- C6 pad 2: Net-(C6-Pad2) -> GND
- C8 pad 1: GND -> Net-(C6-Pad1)
- C8 pad 2: Net-(C8-Pad2) -> GND
- C9 pad 2: +12V -> Net-(C9-Pad2)
- D3 pad 1: Net-(C14-Pad1) -> GND
- D3 pad 2: +12V -> Net-(D3-Pad2)
- D4 pad 1: GND -> Net-(C2-Pad1)
- D4 pad 2: Net-(D4-Pad2) -> Net-(C4-Pad2)
- D5 pad 1: Net-(C11-Pad1) -> GND
- D5 pad 2: +4V -> Net-(D5-Pad2)
- D6 pad 1: Net-(C12-Pad1) -> Net-(C13-Pad1)
- D6 pad 2: +4V -> Net-(C6-Pad1)
- D7 pad 1: Net-(C13-Pad1) -> Net-(C14-Pad1)
- D7 pad 2: +4V -> Net-(C6-Pad1)
- J2 pad 1: Net-(J2-Pad1) -> Net-(C4-Pad2)
- J2 pad 2: Net-(C11-Pad1) -> GND
- J4 pad 1: +12V -> Net-(J4-Pad1)
- J4 pad 2: GND -> Net-(J4-Pad2)
- J5 pad 2: Net-(C12-Pad1) -> Net-(J5-Pad2)
- J5 pad 5: Net-(J5-Pad5) -> GND
- J5 pad 6: GND -> Net-(J5-Pad6)
- R1 pad 1: Net-(C11-Pad1) -> Net-(C13-Pad1)
- R10 pad 1: Net-(R10-Pad1) -> Net-(C10-Pad2)
- R10 pad 2: Net-(J5-Pad7) -> Net-(J4-Pad1)
- R11 pad 1: Net-(R11-Pad1) -> Net-(C11-Pad2)
- R11 pad 2: Net-(J5-Pad5) -> Net-(J4-Pad2)
- R12 pad 1: Net-(R12-Pad1) -> Net-(C12-Pad2)
- R12 pad 2: Net-(J5-Pad3) -> Net-(J4-Pad3)
- R13 pad 2: Net-(J5-Pad1) -> Net-(J5-Pad2)
- R14 pad 2: Net-(J5-Pad4) -> Net-(J5-Pad3)
- R15 pad 2: Net-(J5-Pad8) -> Net-(J5-Pad1)
- R18 pad 1: +4V -> Net-(R18-Pad1)
- R18 pad 2: Net-(D4-Pad2) -> Net-(R18-Pad2)
- R19 pad 2: Net-(R19-Pad2) -> Net-(Q1-Pad1)
- R4 pad 1: Net-(J2-Pad1) -> Net-(D3-Pad2)
- R4 pad 2: Net-(C1-Pad1) -> Net-(R4-Pad2)
- R5 pad 1: Net-(C5-Pad2) -> Net-(J1-Pad1)
- R5 pad 2: Net-(J3-Pad3) -> Net-(C1-Pad1)
- R6 pad 1: Net-(C6-Pad2) -> Net-(C6-Pad1)
- R6 pad 2: Net-(J3-Pad2) -> Net-(D5-Pad2)
- R7 pad 1: Net-(C7-Pad2) -> Net-(C5-Pad2)
- R8 pad 1: Net-(C8-Pad2) -> Net-(C7-Pad2)
- R8 pad 2: Net-(J4-Pad3) -> Net-(J3-Pad2)
- R9 pad 1: Net-(R9-Pad1) -> Net-(C9-Pad2)
- R9 pad 2: Net-(J5-Pad9) -> Net-(J3-Pad3)
- U1 pad 1: Net-(D4-Pad2) -> Net-(D5-Pad2)
- U1 pad 2: +4V -> Net-(C6-Pad1)
- U1 pad 3: Net-(C14-Pad1) -> Net-(C2-Pad1)
- U2 pad 1: Net-(J2-Pad1) -> Net-(J1-Pad1)
- U2 pad 10: Net-(R11-Pad1) -> Net-(R22-Pad1)
- U2 pad 11: Net-(C5-Pad2) -> Net-(C9-Pad2)
- U2 pad 13: Net-(C11-Pad1) -> Net-(C13-Pad1)
- U2 pad 14: Net-(C6-Pad2) -> Net-(C10-Pad2)
- U2 pad 15: Net-(C7-Pad2) -> Net-(R15-Pad1)
- U2 pad 16: Net-(C8-Pad2) -> Net-(C11-Pad2)
- U2 pad 17: Net-(R14-Pad1) -> Net-(C12-Pad2)
- U2 pad 18: Net-(R12-Pad1) -> Net-(R20-Pad1)
- U2 pad 19: Net-(U2-Pad19) -> Net-(R19-Pad1)
- U2 pad 20: Net-(C10-Pad1) -> Net-(C15-Pad1)
- U2 pad 22: Net-(R10-Pad1) -> Net-(R14-Pad1)
- U2 pad 23: Net-(R9-Pad1) -> Net-(U2-Pad23)
- U2 pad 24: Net-(R19-Pad2) -> Net-(R18-Pad2)
- U2 pad 28: Net-(C11-Pad1) -> Net-(C13-Pad1)
- U2 pad 4: Net-(J2-Pad4) -> Net-(J1-Pad4)
- U2 pad 5: Net-(J2-Pad5) -> Net-(J1-Pad5)
- U2 pad 6: Net-(U2-Pad6) -> Net-(C5-Pad2)
- U2 pad 7: Net-(U2-Pad7) -> Net-(C7-Pad2)
- U2 pad 9: Net-(R15-Pad1) -> Net-(R4-Pad2)
- U3 pad 1: Net-(C13-Pad1) -> Net-(C14-Pad1)
- U3 pad 13: GND -> Net-(C14-Pad2)
- U3 pad 15: Net-(R19-Pad1) -> Net-(R18-Pad1)
- U3 pad 18: GND -> Net-(C14-Pad2)
- U3 pad 2: Net-(C13-Pad1) -> Net-(C14-Pad1)
- U3 pad 6: Net-(U3-Pad6) -> Net-(C14-Pad2)
- U3 pad 9: GND -> Net-(C14-Pad2)
Routing:
- net +12V: track 108.7 -> 0.00 mm
- net Net-(J2-Pad1): track 40.8 -> 0.00 mm
- net Net-(C11-Pad1): track 39.6 -> 0.00 mm
- net Net-(C12-Pad1): track 38.0 -> 0.00 mm
- net +4V: track 37.9 -> 0.00 mm
- net GND: track 35.8 -> 0.00 mm, vias 12 -> 0
- net Net-(C5-Pad2): track 35.4 -> 0.00 mm, vias 2 -> 0
- net Net-(R15-Pad1): track 34.6 -> 0.00 mm, vias 2 -> 0
- net Net-(R19-Pad1): track 33.7 -> 0.00 mm, vias 2 -> 0
- net Net-(R10-Pad1): track 30.9 -> 0.00 mm, vias 2 -> 0
- net Net-(R9-Pad1): track 30.0 -> 0.00 mm, vias 2 -> 0
- net Net-(R17-Pad2): track 29.8 -> 0.00 mm, vias 2 -> 0
- net Net-(R16-Pad2): track 26.3 -> 0.00 mm, vias 2 -> 0
- net Net-(J5-Pad5): track 25.1 -> 0.00 mm
- net Net-(C6-Pad2): track 23.2 -> 0.00 mm, vias 2 -> 0
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- removed copper zone on F.Cu, net (none)
- removed copper zone on B.Cu, net GND
Other:
- board size 50 x 50 mm -> 80 x 70 mm
- board text removed: "+12"
- board text removed: "Antena Mantener libre"
- board text removed: "DomIO32"
- board text removed: "E1"
- board text removed: "E2"
- board text removed: "E3"
- board text removed: "E4"
- board text removed: "Estado"
- board text removed: "Expansion"
- board text removed: "G"
- board text removed: "HECHO EN ARGENTINA"
- board text removed: "Modo"
- board text removed: "PGM"
- board text removed: "Reset"
- board text removed: "WGP"

Commit message: Nuevo circuito co relees
Nuevo circuito co relees
Parts:
- added C16: 100uf / 16v, Capacitor_THT:CP_Radial_D6.3mm_P2.50mm, F.Cu at (145.0, 88.5)
- added C17: 100uf / 16v, Capacitor_THT:CP_Radial_D6.3mm_P2.50mm, F.Cu at (145.0, 80.5)
- C1, C10, C11, C12, C13, C4, C5, C7, C8, C9, R10, R11, R12, R6, R7, R8, R9, U1: moved to B.Cu
- moved R15 106.8 mm to (116.0, 64.5), turned to 180 degrees
- moved R13 104.6 mm to (116.0, 67.5), turned to 180 degrees
- moved R2 103.8 mm to (137.0, 48.0), turned to 90 degrees
- moved R3 101.4 mm to (117.0, 48.0), turned to 90 degrees
- moved R5 100.5 mm to (114.0, 48.0), turned to 90 degrees
- moved R1 95.6 mm to (111.0, 48.0), turned to 90 degrees
- moved R4 90.4 mm to (147.0, 48.0), turned to 90 degrees
- moved C1 89.2 mm to (127.0, 48.0), turned to 90 degrees
- moved J1 87.6 mm to (184.5, 82.0), turned to 270 degrees
- moved R14 86.3 mm to (116.0, 70.5), turned to 180 degrees
- moved C4 83.1 mm to (114.5, 104.5), turned to 180 degrees
- moved Q1 82.1 mm to (124.0, 75.0)
- moved R21 78.2 mm to (152.5, 75.0), turned to 90 degrees
- moved R22 76.3 mm to (168.5, 75.0), turned to 90 degrees
- moved C15 73.5 mm to (162.0, 82.0)
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Other:
- board size 80 x 70 mm -> 80 x 65 mm

Commit message: Reestructuracion del proyecto
Reestructuracion del proyecto
Parts:
- removed the R15 at (116.0, 64.5)
- J5: value USB_B_Micro -> Conn_01x03; footprint Connector_USB:USB_Micro-B_GCT_USB3076-30-A -> Connector_PinHeader_2.54mm:PinHeader_1x03_P2.54mm_Vertical
- moved J5 7.02 mm to (110.0, 60.5), turned to 0 degrees
- renumbered C16 to C14, C17 to C15, C14 to C16, C15 to C17, R14 to R13, R13 to R14, R16 to R15, R17 to R16, R18 to R17, R19 to R18, R20 to R19, R21 to R20, R22 to R21
Connections:
- J5 pad 1: Net-(J5-Pad1) -> GND
- R13 pad 1: Net-(R14-Pad1) -> Net-(R13-Pad1)
- R14 pad 1: Net-(R13-Pad1) -> Net-(R14-Pad1)
- R18 pad 1: Net-(R19-Pad1) -> Net-(R18-Pad1)
- R19 pad 1: Net-(R20-Pad1) -> Net-(R19-Pad1)
- R20 pad 1: Net-(R21-Pad1) -> Net-(R20-Pad1)
- R21 pad 1: Net-(R22-Pad1) -> Net-(R21-Pad1)
- U2 pad 10: Net-(R22-Pad1) -> Net-(R13-Pad1)
- U2 pad 12: Net-(R21-Pad1) -> Net-(R4-Pad2)
- U2 pad 18: Net-(R20-Pad1) -> Net-(R21-Pad1)
- U2 pad 19: Net-(R19-Pad1) -> Net-(R20-Pad1)
- U2 pad 21: Net-(R13-Pad1) -> Net-(R19-Pad1)
- U2 pad 22: Net-(R14-Pad1) -> Net-(R18-Pad1)
- U2 pad 9: Net-(R4-Pad2) -> Net-(R14-Pad1)

Commit message: Correcciones al circuito y avance con la placa
Correcciones al circuito y avance con la placa
Parts:
- moved J1 7.02 mm to (184.0, 75.0), turned to 0 degrees
- moved R13 4.92 mm to (114.0, 66.0)
- moved R14 4.92 mm to (114.0, 63.0)
- moved D10 2.00 mm to (160.0, 75.0)
- moved D11 2.00 mm to (176.0, 75.0)
- moved D8 2.00 mm to (128.0, 75.0)
- moved D9 2.00 mm to (144.0, 75.0)
- moved K1 2.00 mm to (128.0, 71.0)
- moved K2 2.00 mm to (144.0, 71.0)
- moved K3 2.00 mm to (160.0, 71.0)
- moved K4 2.00 mm to (176.0, 71.0)
- moved Q1 2.00 mm to (122.0, 75.0)
- moved Q2 2.00 mm to (138.0, 75.0)
- moved Q3 2.00 mm to (154.0, 75.0)
- moved Q4 2.00 mm to (170.0, 75.0)
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Connections:
- C2 pad 1: Net-(C2-Pad1) -> +12V
- C3 pad 1: Net-(C2-Pad1) -> +12V
- D4 pad 1: Net-(C2-Pad1) -> +12V
- D8 pad 1: Net-(C2-Pad1) -> +12V
- K1 pad 12: Net-(K1-Pad12) -> unconnected-(K1-Pad12)
- K1 pad A1: Net-(C2-Pad1) -> +12V
- K2 pad 12: Net-(K2-Pad12) -> unconnected-(K2-Pad12)
- K3 pad 12: Net-(K3-Pad12) -> unconnected-(K3-Pad12)
- K4 pad 12: Net-(K4-Pad12) -> unconnected-(K4-Pad12)
- U1 pad 3: Net-(C2-Pad1) -> +12V
- U2 pad 15: Net-(U2-Pad15) -> unconnected-(U2-Pad15)
- U2 pad 23: Net-(U2-Pad23) -> unconnected-(U2-Pad23)
- U3 pad 10: Net-(U3-Pad10) -> unconnected-(U3-Pad10)
- U3 pad 14: Net-(U3-Pad14) -> unconnected-(U3-Pad14)
- U3 pad 16: Net-(U3-Pad16) -> unconnected-(U3-Pad16)
- U3 pad 17: Net-(U3-Pad17) -> unconnected-(U3-Pad17)
- U3 pad 3: Net-(U3-Pad3) -> unconnected-(U3-Pad3)
- U3 pad 4: Net-(U3-Pad4) -> unconnected-(U3-Pad4)
- U3 pad 5: Net-(U3-Pad5) -> unconnected-(U3-Pad5)
- U3 pad 7: Net-(U3-Pad7) -> unconnected-(U3-Pad7)
- U3 pad 8: Net-(U3-Pad8) -> unconnected-(U3-Pad8)
Routing:
- net Net-(J7-Pad1): track 0.00 -> 106.1 mm
- net +12V: track 0.00 -> 55.5 mm
- net Net-(J6-Pad3): track 0.00 -> 33.0 mm
- net Net-(J6-Pad2): track 0.00 -> 21.7 mm
- net Net-(J7-Pad2): track 0.00 -> 12.7 mm
- net Net-(J6-Pad1): track 0.00 -> 11.3 mm
Other:
- net class 0,25 removed
- net class 1 removed
- net class Default removed

Commit message: PCB
PCB
Parts:
- moved C8 4.03 mm to (128.0, 90.0)
Routing:
- net +12V: track 55.5 -> 112.5 mm
- net Net-(C6-Pad1): track 0.00 -> 30.2 mm
- net Net-(R17-Pad2): track 0.00 -> 20.5 mm, vias 0 -> 1
- net Net-(D5-Pad2): track 0.00 -> 17.1 mm, vias 0 -> 1
- net Net-(R15-Pad2): track 0.00 -> 13.8 mm, vias 0 -> 1
- net Net-(C4-Pad2): track 0.00 -> 12.1 mm
- net Net-(C1-Pad1): track 0.00 -> 10.7 mm
- net Net-(D11-Pad2): track 0.00 -> 10.4 mm
- net Net-(D9-Pad2): track 0.00 -> 10.4 mm
- net Net-(D10-Pad2): track 0.00 -> 10.4 mm
- net Net-(D8-Pad2): track 0.00 -> 10.4 mm
- net Net-(R16-Pad2): track 0.00 -> 10.2 mm, vias 0 -> 1
- net Net-(C9-Pad2): track 0.00 -> 9.34 mm
- net Net-(C7-Pad2): track 0.00 -> 9.34 mm
- net Net-(C5-Pad2): track 0.00 -> 9.34 mm
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
Commit message: PCB
PCB
Parts:
- added R22: 22R, Resistor_SMD:R_0805_2012Metric_Pad1.20x1.40mm_HandSolder, F.Cu at (114.0, 60.0)
- J5: value Conn_01x03 -> Conn_01x04; footprint Connector_PinHeader_2.54mm:PinHeader_1x03_P2.54mm_Vertical -> Connector_PinHeader_2.54mm:PinHeader_1x04_P2.54mm_Vertical
- moved J1 10.3 mm to (183.5, 85.3), turned to 180 degrees
- moved C17 3.24 mm to (163.2, 85.0)
Connections:
- C14 pad 2: Net-(C14-Pad2) -> GND
- C16 pad 2: Net-(C14-Pad2) -> GND
- J5 pad 1: GND -> Net-(J5-Pad1)
- R13 pad 2: Net-(J5-Pad3) -> Net-(J5-Pad2)
- R14 pad 2: Net-(J5-Pad2) -> Net-(J5-Pad3)
- R18 pad 1: Net-(R18-Pad1) -> Net-(U2-Pad18)
- R19 pad 1: Net-(R19-Pad1) -> Net-(U2-Pad19)
- R20 pad 1: Net-(R20-Pad1) -> Net-(U2-Pad21)
- R21 pad 1: Net-(R21-Pad1) -> Net-(U2-Pad22)
- U2 pad 11: Net-(C9-Pad2) -> Net-(C7-Pad2)
- U2 pad 14: Net-(C10-Pad2) -> Net-(C5-Pad2)
- U2 pad 15: unconnected-(U2-Pad15) -> Net-(R22-Pad1)
- U2 pad 18: Net-(R21-Pad1) -> Net-(U2-Pad18)
- U2 pad 19: Net-(R20-Pad1) -> Net-(U2-Pad19)
- U2 pad 21: Net-(R19-Pad1) -> Net-(U2-Pad21)
- U2 pad 22: Net-(R18-Pad1) -> Net-(U2-Pad22)
- U2 pad 6: Net-(C5-Pad2) -> Net-(C10-Pad2)
- U2 pad 7: Net-(C7-Pad2) -> Net-(C9-Pad2)
- U3 pad 13: Net-(C14-Pad2) -> GND
- U3 pad 18: Net-(C14-Pad2) -> GND
- U3 pad 6: Net-(C14-Pad2) -> GND
- U3 pad 9: Net-(C14-Pad2) -> GND
Routing:
- net Net-(C13-Pad1): track 0.00 -> 81.9 mm, vias 0 -> 2
- net Net-(R22-Pad1): track 0.00 -> 65.7 mm, vias 0 -> 1
- net Net-(R14-Pad1): track 0.00 -> 65.6 mm, vias 0 -> 1
- net Net-(R13-Pad1): track 0.00 -> 60.6 mm, vias 0 -> 1
- net Net-(C14-Pad1): track 0.00 -> 54.6 mm, vias 0 -> 1
- net Net-(U2-Pad18): track 0.00 -> 53.0 mm, vias 0 -> 1
- net Net-(J1-Pad5): track 0.00 -> 44.8 mm, vias 0 -> 1
- net Net-(J1-Pad1): track 0.00 -> 43.8 mm
- net Net-(J1-Pad4): track 0.00 -> 43.6 mm, vias 0 -> 1
- net Net-(U2-Pad19): track 0.00 -> 38.8 mm, vias 0 -> 1
- net Net-(C5-Pad2): track 9.34 -> 45.2 mm
- net +12V: track 112.5 -> 147.5 mm
- net Net-(R3-Pad2): track 0.00 -> 29.6 mm, vias 0 -> 1
- net Net-(R4-Pad2): track 0.00 -> 27.6 mm, vias 0 -> 1
- net Net-(C7-Pad2): track 9.34 -> 35.8 mm
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
Commit message: Antes de agregar areas de relleno
Antes de agregar areas de relleno
Parts:
- moved SW1 7.91 mm to (130.5, 50.5), turned to 180 degrees
- moved D1 0.50 mm to (134.5, 48.0), turned to 90 degrees
- moved R2 0.50 mm to (137.5, 48.0), turned to -90 degrees
- turned D2 to 90 degrees
- turned R3 to -90 degrees
- turned C1 to -90 degrees
- turned D3 to 90 degrees
- turned R4 to -90 degrees
Routing:
- net Net-(J1-Pad1): track 43.8 -> 135.4 mm, vias 0 -> 3
- net Net-(R4-Pad2): track 27.6 -> 112.3 mm, vias 1 -> 3
- net Net-(R2-Pad2): track 26.2 -> 104.2 mm, vias 1 -> 3
- net Net-(C13-Pad1): track 81.9 -> 144.2 mm
- net Net-(R3-Pad2): track 29.6 -> 91.8 mm, vias 1 -> 3
- net Net-(C1-Pad1): track 10.7 -> 21.6 mm
- net Net-(J5-Pad1): track 0.00 -> 3.21 mm
- net Net-(C11-Pad2): track 33.4 -> 34.4 mm
- net Net-(C12-Pad2): track 26.0 -> 27.0 mm

Commit message: Final PCB
Final PCB
Parts:
- moved R13 3.00 mm to (114.0, 63.0)
- moved R14 3.00 mm to (114.0, 66.0)
Connections:
- U2 pad 10: Net-(R13-Pad1) -> Net-(R14-Pad1)
- U2 pad 9: Net-(R14-Pad1) -> Net-(R13-Pad1)
Routing:
- net Net-(R13-Pad1): track 60.6 -> 65.8 mm
- net Net-(R14-Pad1): track 65.6 -> 61.5 mm
- net Net-(R4-Pad2): track 112.3 -> 115.4 mm
- net Net-(J1-Pad1): track 135.4 -> 133.0 mm
- net Net-(R2-Pad2): track 104.2 -> 106.0 mm
- net Net-(J1-Pad4): track 43.6 -> 42.1 mm
- net Net-(J1-Pad5): track 44.8 -> 43.2 mm
- net Net-(C13-Pad1): track 144.2 -> 145.6 mm
- net Net-(C5-Pad2): track 45.2 -> 44.1 mm
- net Net-(C12-Pad2): track 27.0 -> 25.9 mm
- net Net-(C11-Pad2): track 34.4 -> 33.6 mm
- net Net-(R22-Pad1): track 65.7 -> 66.5 mm
- net Net-(D5-Pad2): track 16.8 -> 16.1 mm
- net Net-(R3-Pad2): track 91.8 -> 92.5 mm
- net +12V: track 147.5 -> 148.1 mm
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- added copper zone on B.Cu, net GND
- added copper zone on F.Cu, net GND
Other:
- board text added: "Dom32-IO-WiFi"
- board text added: "WGP 2022"
