File: Circuito/DomIO32.kicad_pcb (KiCad board)
At the start: 2 copper layers, 80 x 65 mm, 69 parts, among them J1 Conector 1x5, J2 Bornera x2, J3 Bornera x3, J4 Bornera x3, J5 Conn_01x04, J6 Bornera x3, J7 Bornera x2, K1 FINDER-36.11, K2 FINDER-36.11, K3 FINDER-36.11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

Commit message: Versión revisada para solicitud de cotización
Versión revisada para solicitud de cotización
Routing:
- net Net-(J7-Pad2): track 12.7 -> 11.0 mm
- net Net-(J6-Pad3): track 33.0 -> 32.1 mm
- net Net-(R19-Pad1): track 38.8 -> 37.9 mm
- net Net-(R13-Pad1): track 65.8 -> 65.0 mm
- net Net-(R14-Pad1): track 61.5 -> 60.9 mm
- net (no net): vias 0 -> 6
Other:
- board text added: "(+)"
- board text added: "(-)"
- board text added: "ANTENA"
- board text added: "AUX"
- board text added: "COMUN"
- board text added: "DEBUG"
- board text added: "ESTADO"
- board text added: "ICSP"
- board text added: "IO1"
- board text added: "IO2"
- board text added: "IO3"
- board text added: "IO4"
- board text added: "IO5"
- board text added: "IO6"
- board text added: "MODO"
- board text added: "RESET"
- board text added: "SALIDAS"
