File: Circuito/DomIO32.kicad_pcb (KiCad board)
At the start: 2 copper layers, 80 x 65 mm, 69 parts, among them J1 Conector 1x5, J2 Bornera x2, J3 Bornera x3, J4 Bornera x3, J5 Conn_01x04, J6 Bornera x3, J7 Bornera x2, K1 FINDER-36.11, K2 FINDER-36.11, K3 FINDER-36.11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

Commit message: MicroSD agregada
MicroSD agregada
Parts:
- removed R22: 22R, Resistor_SMD:R_0805_2012Metric_Pad1.20x1.40mm_HandSolder
- added J8: MEM2067-02-180-00-A, Connector_Card:microSD_HC_Wuerth_693072010801, F.Cu at (173.1, 87.1)
- added R23: 1K, Resistor_SMD:R_0805_2012Metric_Pad1.20x1.40mm_HandSolder, B.Cu at (165.8, 84.2)
- added R24: 1K, Resistor_SMD:R_0805_2012Metric_Pad1.20x1.40mm_HandSolder, B.Cu at (172.8, 84.2)
- added R25: 1K, Resistor_SMD:R_0805_2012Metric_Pad1.20x1.40mm_HandSolder, B.Cu at (169.0, 84.2)
- added R26: 1K, Resistor_SMD:R_0805_2012Metric_Pad1.20x1.40mm_HandSolder, B.Cu at (176.2, 83.2)
- added R27: 10K, Resistor_SMD:R_0805_2012Metric_Pad1.20x1.40mm_HandSolder, F.Cu at (168.5, 99.2)
- added R28: 10K, Resistor_SMD:R_0805_2012Metric_Pad1.20x1.40mm_HandSolder, F.Cu at (170.8, 99.2)
- added R29: 10K, Resistor_SMD:R_0805_2012Metric_Pad1.20x1.40mm_HandSolder, F.Cu at (175.0, 99.2)
- added R30: 10K, Resistor_SMD:R_0805_2012Metric_Pad1.20x1.40mm_HandSolder, F.Cu at (177.2, 99.2)
- C3: value 1000uf / 50v -> 1000uf / 25v
- C6: value 100uf / 16v -> 100uf / 25v
- D10, D11, D5, D8, D9: value LL4148 -> LL4148-GS08
- D4, D6, D7: value M7 -> 3191-M7CT-ND
- J1: value Conector 1x5 -> Poste X 5
- J2, J7: value Bornera x2 -> 277-1667-ND
- J3, J4, J6: value Bornera x3 -> 277-1578-ND
- J5: value Conn_01x04 -> Poste X 2; footprint Connector_PinHeader_2.54mm:PinHeader_1x04_P2.54mm_Vertical -> Connector_PinHeader_2.54mm:PinHeader_1x02_P2.54mm_Vertical
- K1, K2, K3, K4: value FINDER-36.11 -> AZ943-1CH-12DE
- Q1, Q2, Q3, Q4: value BC848 -> BC847C-TP
- R13: value 22R -> 0R
- R14: value 22R -> 33R
- R15, R16, R17: moved to B.Cu
- U1: value LM1117-3.3 -> ZLDO1117QG33TADICT-ND
- U3: value ESP-02 -> 1965-ESP-WROOM-02D-N4CT-ND
- moved R13 35.1 mm to (133.8, 92.0), turned to -90 degrees
- moved C16 20.8 mm to (154.2, 102.2)
- moved R17 11.2 mm to (163.8, 94.5), turned to 180 degrees
- moved R15 11.1 mm to (163.8, 99.5), turned to 180 degrees
- moved R16 7.27 mm to (163.8, 97.0), turned to 180 degrees
- moved R14 5.52 mm to (114.5, 60.5)
- moved C17 2.34 mm to (161.0, 84.2), turned to 180 degrees
Connections:
- C6 pad 1: Net-(C6-Pad1) -> Net-(U1-VO)
- C8 pad 1: Net-(C6-Pad1) -> Net-(U1-VO)
- D6 pad 2: Net-(C6-Pad1) -> Net-(D6-A)
- D7 pad 2: Net-(C6-Pad1) -> Net-(D6-A)
- J5 pad 1: Net-(J5-Pad1) -> Net-(J5-Pin_1)
- J5 pad 2: Net-(J5-Pad2) -> GND
- R13 pad 1: Net-(R13-Pad1) -> Net-(D6-A)
- R13 pad 2: Net-(J5-Pad2) -> Net-(U1-VO)
- R14 pad 2: Net-(J5-Pad3) -> Net-(J5-Pin_1)
- R6 pad 1: Net-(C6-Pad1) -> Net-(U1-VO)
- U1 pad 2: Net-(C6-Pad1) -> Net-(U1-VO)
- U2 pad 9: Net-(R13-Pad1) -> Net-(U2-OSC1/RP3/RA2)
Routing:
- net Net-(R13-Pad1): track 65.0 -> 0.00 mm, vias 1 -> 0
- net Net-(U2-Vbus/RB6): track 66.2 -> 17.7 mm, vias 1 -> 0
- net Net-(U2-OSC1/RP3/RA2): track 0.00 -> 35.2 mm, vias 0 -> 2
- net Net-(C6-Pad1): track 30.2 -> 0.00 mm
- net Net-(D6-K): track 145.6 -> 169.6 mm
- net Net-(U1-VO): track 0.00 -> 21.9 mm
- net Net-(J8-DAT3/CD): track 0.00 -> 21.6 mm, vias 0 -> 1
- net Net-(U2-RP15/RB13): track 20.0 -> 3.51 mm, vias 1 -> 0
- net Net-(U3-RESET): track 2.74 -> 18.0 mm, vias 1 -> 0
- net Net-(J8-DAT0): track 0.00 -> 14.5 mm, vias 0 -> 1
- net Net-(J1-Pin_5): track 43.2 -> 57.5 mm, vias 1 -> 2
- net Net-(U3-TXD): track 3.36 -> 14.7 mm, vias 1 -> 0
- net Net-(J8-DAT2): track 0.00 -> 9.98 mm
- net Net-(J8-DAT1): track 0.00 -> 9.65 mm
- net Net-(U3-RXD): track 2.74 -> 11.5 mm, vias 1 -> 0
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