File: Circuito/DomIO32.kicad_sch (KiCad schematic)
At the start: 68 parts, among them J1 Conector 1x5, J2 Bornera x2, J3 Bornera x3, J4 Bornera x3, J5 Conn_01x03, J6 Bornera x3, J7 Bornera x2, K1 FINDER-36.11, K2 FINDER-36.11, K3 FINDER-36.11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

Commit message: PCB
PCB
Parts:
- removed J5: Conn_01x03, Connector_PinHeader_2.54mm:PinHeader_1x03_P2.54mm_Vertical, symbol Connector_Generic:Conn_01x03
- added J5: Conn_01x04, Connector_PinHeader_2.54mm:PinHeader_1x04_P2.54mm_Vertical, symbol Connector_Generic:Conn_01x04
- added R22: 22R, Resistor_SMD:R_0805_2012Metric_Pad1.20x1.40mm_HandSolder, symbol Device:R
Connections:
- net GND: now also C14.2, C16.2, U3.13 (GND), U3.18 (GND), U3.6 (IO15), U3.9 (GND), J5.4 (Pin_4)
- net at C9.2, R9.1: now also U2.7 (TDI/RP9/RB3); no longer U2.11 (SOSCI/RP10/RB4)
- net at C10.2, R10.1: now also U2.6 (RP8/RB2); no longer U2.14 (PGED3/RP11/RB5)
- net at R21.1: now also U2.22 (D+/RB11); no longer U2.18 (TMS/RP14/RB9)
- net at R20.1: now also U2.21 (D-/RB10); no longer U2.19 (PGEC3/RP18/RC9)
- net at R19.1: now also U2.19 (PGEC3/RP18/RC9); no longer U2.21 (D-/RB10)
- net at R18.1: now also U2.18 (TMS/RP14/RB9); no longer U2.22 (D+/RB11)
- net at R14.2: now also J5.3 (Pin_3)
- net at R13.2: now also J5.2 (Pin_2)
- net at U2.15 (Vbus/RB6): now also R22.1
- net at C5.2, R7.1: now also U2.14 (PGED3/RP11/RB5); no longer U2.6 (RP8/RB2)
- net at C7.2, R8.1: now also U2.11 (SOSCI/RP10/RB4); no longer U2.7 (TDI/RP9/RB3)
- new net: J5.1 (Pin_1), R22.2

Commit message: Final PCB
Final PCB
Connections:
- net at U2.10 (OSC2/RP4/RA3): now also R14.1; no longer R13.1
- net at U2.9 (OSC1/RP3/RA2): now also R13.1; no longer R14.1
Changed lines of the file:
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@@
-    (stroke (width 0) (type default) (color 0 0 0 0))
-  )
-  (wire (pts (xy 86.36 93.98) (xy 86.36 116.84))
     (stroke (width 0) (type default) (color 0 0 0 0))
   )
@@
     (stroke (width 0) (type default) (color 0 0 0 0))
   )
+  (wire (pts (xy 86.36 96.52) (xy 86.36 116.84))
+    (stroke (width 0) (type default) (color 0 0 0 0))
+  )
   (wire (pts (xy 45.72 73.66) (xy 45.72 78.74))
     (stroke (width 0) (type default) (color 0 0 0 0))
@@
     (stroke (width 0) (type default) (color 0 0 0 0))
   )
-  (wire (pts (xy 87.63 96.52) (xy 88.9 96.52))
-    (stroke (width 0) (type default) (color 0 0 0 0))
-  )
   (wire (pts (xy 40.64 105.41) (xy 40.64 113.03))
     (stroke (width 0) (type default) (color 0 0 0 0))
@@
     (stroke (width 0) (type default) (color 0 0 0 0))
   )
-  (wire (pts (xy 87.63 114.3) (xy 87.63 96.52))
-    (stroke (width 0) (type default) (color 0 0 0 0))
-  )
   (wire (pts (xy 81.28 149.86) (xy 106.68 149.86))
     (stroke (width 0) (type default) (color 0 0 0 0))
@@
     (stroke (width 0) (type default) (color 0 0 0 0))
   )
+  (wire (pts (xy 88.9 96.52) (xy 86.36 96.52))
+    (stroke (width 0) (type default) (color 0 0 0 0))
+  )
   (wire (pts (xy 203.2 107.95) (xy 203.2 106.68))
     (stroke (width 0) (type default) (color 0 0 0 0))
@@
     (stroke (width 0) (type default) (color 0 0 0 0))
   )
-  (wire (pts (xy 88.9 93.98) (xy 86.36 93.98))
-    (stroke (width 0) (type default) (color 0 0 0 0))
-  )
   (wire (pts (xy 203.2 82.55) (xy 203.2 81.28))
     (stroke (width 0) (type default) (color 0 0 0 0))
@@
     (stroke (width 0) (type default) (color 0 0 0 0))
   )
+  (wire (pts (xy 87.63 93.98) (xy 87.63 114.3))
+    (stroke (width 0) (type default) (color 0 0 0 0))
+  )
   (wire (pts (xy 204.47 55.88) (xy 204.47 40.64))
     (stroke (width 0) (type default) (color 0 0 0 0))
@@
     (stroke (width 0) (type default) (color 0 0 0 0))
   )
+  (wire (pts (xy 88.9 93.98) (xy 87.63 93.98))
+    (stroke (width 0) (type default) (color 0 0 0 0))
+  )
